File: Tarea3/PLC4UNI/ENERGY-METER.kicad_sch (KiCad schematic)
At the start: 0 parts

Commit message: Cambio de directorio [Tarea2->CAD]
Changed lines of the file:
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@@
 	(hierarchical_label "TX"
 		(shape output)
-		(at 110.49 69.85 0)
+		(at 208.28 73.66 0)
 		(effects
 			(font
@@
 	(hierarchical_label "RX"
 		(shape output)
-		(at 110.49 66.04 0)
+		(at 208.28 69.85 0)
 		(effects
 			(font
