File: Tarea3/PLC4UNI/plcuni_top.kicad_sch (KiCad schematic)
At the start: 0 parts

Commit message: Cambio de directorio [Tarea2->CAD]
Parts:
- added C38: C_0603, PCM_Capacitor_SMD_AKL:C_0603_1608Metric, symbol PCM_Capacitor_US_AKL:C_0603
- added R53: R_0603, PCM_Resistor_SMD_AKL:R_0603_1608Metric, symbol PCM_Resistor_US_AKL:R_0603
- added R54, R55: 0R, PCM_Resistor_SMD_AKL:R_0603_1608Metric, symbol PCM_Resistor_US_AKL:R_0603
- added TP4, TP5, TP6, TP7: TestPoint, symbol Connector:TestPoint
- added U18: ESP32-S3-WROOM-1, Espressif:ESP32-S3-WROOM-1, symbol Espressif:ESP32-S3-WROOM-1
- added U19: ADS1115IDGS, Package_SO:TSSOP-10_3x3mm_P0.5mm, symbol Analog_ADC:ADS1115IDGS
Connections:
- net IN-0-10V/OUT3V3: now also TP6.1, U19.6 (AIN2)
- net IN-0-10V1/OUT3V3: now also TP7.1, U19.7 (AIN3)
- net IN-4-20MA/OUT: now also TP4.1, U19.4 (AIN0)
- net IN-4-20MA1/OUT: now also TP5.1, U19.5 (AIN1)
- new net 3.3V: R53.1, U18.2 (3V3)
- new net EMRX: U18.36 (U0RXD/GPIO44/CLK_OUT2)
- new net EM_TX: U18.37 (U0TXD/GPIO43/CLK_OUT1)
- new net EN: C38.1, R53.2, U18.3 (EN)
- new net GND: C38.2, U18.1 (GND), U18.40 (GND), U18.41 (GND)
- new net I2C_SCK: U18.11 (GPIO18/U1RXD/ADC2_CH7/CLK_OUT3)
- new net I2C_SDA: U18.10 (GPIO17/U1TXD/ADC2_CH6)
- new net IN_NPN1: U18.27 (GPIO0/BOOT)
- new net IN_NPN2: U18.39 (GPIO1/TOUCH1/ADC1_CH0)
- new net IN_NPN3: U18.38 (GPIO2/TOUCH2/ADC1_CH1)
- new net IN_NPN4: U18.15 (GPIO3/TOUCH3/ADC1_CH2)
- new net IN_PNP1: U18.16 (GPIO46)
- new net IN_PNP2: U18.24 (GPIO47/SPICLK_P/SUBSPICLK_P_DIFF)
- new net LCD_CS: U18.35 (MTMS/GPIO42)
- new net LED_INFO: U18.26 (GPIO45)
- new net OUT-PNP/ST1: R54.2
- new net OUT-PNP/ST2: R55.2
- new net OUT_NPN1: U18.4 (GPIO4/TOUCH4/ADC1_CH3)
- new net OUT_NPN2: U18.5 (GPIO5/TOUCH5/ADC1_CH4)
- new net OUT_NPN3: U18.6 (GPIO6/TOUCH6/ADC1_CH5)
- new net OUT_NPN4: U18.7 (GPIO7/TOUCH7/ADC1_CH6)
- new net OUT_PNP1: U18.8 (GPIO15/U0RTS/ADC2_CH4/XTAL_32K_P)
- new net OUT_PNP2: U18.9 (GPIO16/U0CTS/ADC2_CH5/XTAL_32K_N)
- new net OUT_RLY1: U18.23 (GPIO21)
- new net OUT_RLY2: U18.31 (GPIO38/FSPIWP/SUBSPIWP)
- new net RESET: U18.22 (GPIO14/TOUCH14/ADC2_CH3/FSPIWP/FSPIDQS/SUBSPIWP)
- new net RS485-RX: U18.12 (GPIO8/TOUCH8/ADC1_CH7/SUBSPICS1)
- new net RS485-TX: U18.17 (GPIO9/TOUCH9/ADC1_CH8/FSPIHD/SUBSPIHD)
- new net SD_CS: U18.18 (GPIO10/TOUCH10/ADC1_CH9/FSPICS0/FSPIIO4/SUBSPICS0)
- new net SPI_CLK: U18.20 (GPIO12/TOUCH12/ADC2_CH1/FSPICLK/FSPIIO6/SUBSPICLK)
- new net SPI_MISO: U18.21 (GPIO13/TOUCH13/ADC2_CH2/FSPIQ/FSPIIO7/SUBSPIQ)
- new net SPI_MOSI: U18.19 (GPIO11/TOUCH11/ADC2_CH0/FSPID/FSPIIO5/SUBSPID)
- new net ST1_ST2: R54.1, R55.1, U18.32 (MTCK/GPIO39/CLK_OUT3/SUBSPICS1)
- new net TC_FAULT: U18.34 (MTDI/GPIO41/CLK_OUT1)
- new net TEMP_CS: U18.25 (GPIO48/SPICLK_N/SUBSPICLK_N_DIFF)
- new net TP_INT: U18.33 (MTDO/GPIO40/CLK_OUT2)
- new net USB+: U18.14 (GPIO20/U1CTS/ADC2_CH9/CLK_OUT1/USB_D+)
- new net USB-: U18.13 (GPIO19/U1RTS/ADC2_CH8/CLK_OUT2/USB_D-)
Other:
- removed sheet OUT_NPN
- removed sheet OUT_NPN1
- removed sheet OUT_NPN2
- removed sheet OUT_NPN3
- removed sheet OUT_PNP
- added sheet OUT-NPN (OUT-NPN.kicad_sch)
- added sheet OUT-NPN1 (OUT-NPN.kicad_sch)
- added sheet OUT-NPN2 (OUT-NPN.kicad_sch)
- added sheet OUT-NPN3 (OUT-NPN.kicad_sch)
- added sheet OUT-PNP (OUT-PNP.kicad_sch)
- sheet OUT-4-20MA ports: added OUT, ~{ALARM}; removed OUT-4-20MA, /ALARM
