File: PCB/PLC4UNI/IN-0-10V.kicad_sch (KiCad schematic)
At the start: 5 parts

Commit message: add ruteo buck-converter, inputs pnp,npn
Parts:
- renumbered C5 to C9, D5 to D17, D7 to D18, R9 to R23, R11 to R24
Changed lines of the file:
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@@
 		(in_pos_files yes)
 		(dnp no)
-		(property "Reference" "D5"
+		(property "Reference" "D17"
 			(at 100.33 61.1504 90)
 			(show_name no)
@@
 			(project "PLC4UNI"
 				(path "/f171b770-6a1a-4d3a-9dbb-25a622b94557/79ee6e1c-834c-43ff-8dcc-1385cc20b4c2/1a95a96f-95b5-47d3-8bba-4935d279501e"
-					(reference "D5")
-					(unit 1)
-				)
-				(path "/f171b770-6a1a-4d3a-9dbb-25a622b94557/79ee6e1c-834c-43ff-8dcc-1385cc20b4c2/9e9e4298-f102-4294-8a71-c71ffc0789bb"
-					(reference "D6")
+					(reference "D17")
+					(unit 1)
+				)
+				(path "/f171b770-6a1a-4d3a-9dbb-25a622b94557/79ee6e1c-834c-43ff-8dcc-1385cc20b4c2/9e9e4298-f102-4294-8a71-c71ffc0789bb"
+					(reference "D19")
 					(unit 1)
 				)
@@
 		(dnp no)
 		(fields_autoplaced yes)
-		(property "Reference" "#PWR03"
+		(property "Reference" "#PWR042"
 			(at 91.44 66.04 0)
 			(hide yes)
@@
 			(project "PLC4UNI"
 				(path "/f171b770-6a1a-4d3a-9dbb-25a622b94557/79ee6e1c-834c-43ff-8dcc-1385cc20b4c2/1a95a96f-95b5-47d3-8bba-4935d279501e"
-					(reference "#PWR03")
-					(unit 1)
-				)
-				(path "/f171b770-6a1a-4d3a-9dbb-25a622b94557/79ee6e1c-834c-43ff-8dcc-1385cc20b4c2/9e9e4298-f102-4294-8a71-c71ffc0789bb"
-					(reference "#PWR04")
+					(reference "#PWR042")
+					(unit 1)
+				)
+				(path "/f171b770-6a1a-4d3a-9dbb-25a622b94557/79ee6e1c-834c-43ff-8dcc-1385cc20b4c2/9e9e4298-f102-4294-8a71-c71ffc0789bb"
+					(reference "#PWR044")
 					(unit 1)
 				)
@@
 		(dnp no)
 		(fields_autoplaced yes)
-		(property "Reference" "#PWR05"
+		(property "Reference" "#PWR043"
 			(at 120.65 57.15 0)
 			(hide yes)
@@
 			(project "PLC4UNI"
 				(path "/f171b770-6a1a-4d3a-9dbb-25a622b94557/79ee6e1c-834c-43ff-8dcc-1385cc20b4c2/1a95a96f-95b5-47d3-8bba-4935d279501e"
-					(reference "#PWR05")
-					(unit 1)
-				)
-				(path "/f171b770-6a1a-4d3a-9dbb-25a622b94557/79ee6e1c-834c-43ff-8dcc-1385cc20b4c2/9e9e4298-f102-4294-8a71-c71ffc0789bb"
-					(reference "#PWR06")
+					(reference "#PWR043")
+					(unit 1)
+				)
+				(path "/f171b770-6a1a-4d3a-9dbb-25a622b94557/79ee6e1c-834c-43ff-8dcc-1385cc20b4c2/9e9e4298-f102-4294-8a71-c71ffc0789bb"
+					(reference "#PWR045")
 					(unit 1)
 				)
@@
 		(in_pos_files yes)
 		(dnp no)
-		(property "Reference" "C5"
+		(property "Reference" "C9"
 			(at 119.38 85.0899 0)
 			(show_name no)
@@
 			(project "PLC4UNI"
 				(path "/f171b770-6a1a-4d3a-9dbb-25a622b94557/79ee6e1c-834c-43ff-8dcc-1385cc20b4c2/1a95a96f-95b5-47d3-8bba-4935d279501e"
-					(reference "C5")
-					(unit 1)
-				)
-				(path "/f171b770-6a1a-4d3a-9dbb-25a622b94557/79ee6e1c-834c-43ff-8dcc-1385cc20b4c2/9e9e4298-f102-4294-8a71-c71ffc0789bb"
-					(reference "C6")
+					(reference "C9")
+					(unit 1)
+				)
+				(path "/f171b770-6a1a-4d3a-9dbb-25a622b94557/79ee6e1c-834c-43ff-8dcc-1385cc20b4c2/9e9e4298-f102-4294-8a71-c71ffc0789bb"
+					(reference "C10")
 					(unit 1)
 				)
@@
 		(dnp no)
 		(fields_autoplaced yes)
-		(property "Reference" "R11"
+		(property "Reference" "R24"
 			(at 96.52 85.0899 0)
 			(show_name no)
@@
 			(project "PLC4UNI"
 				(path "/f171b770-6a1a-4d3a-9dbb-25a622b94557/79ee6e1c-834c-43ff-8dcc-1385cc20b4c2/1a95a96f-95b5-47d3-8bba-4935d279501e"
-					(reference "R11")
-					(unit 1)
-				)
-				(path "/f171b770-6a1a-4d3a-9dbb-25a622b94557/79ee6e1c-834c-43ff-8dcc-1385cc20b4c2/9e9e4298-f102-4294-8a71-c71ffc0789bb"
-					(reference "R12")
+					(reference "R24")
+					(unit 1)
+				)
+				(path "/f171b770-6a1a-4d3a-9dbb-25a622b94557/79ee6e1c-834c-43ff-8dcc-1385cc20b4c2/9e9e4298-f102-4294-8a71-c71ffc0789bb"
+					(reference "R26")
 					(unit 1)
 				)
@@
 		(dnp no)
 		(fields_autoplaced yes)
-		(property "Reference" "R9"
+		(property "Reference" "R23"
 			(at 82.55 72.39 90)
 			(show_name no)
@@
 			(project "PLC4UNI"
 				(path "/f171b770-6a1a-4d3a-9dbb-25a622b94557/79ee6e1c-834c-43ff-8dcc-1385cc20b4c2/1a95a96f-95b5-47d3-8bba-4935d279501e"
-					(reference "R9")
-					(unit 1)
-				)
-				(path "/f171b770-6a1a-4d3a-9dbb-25a622b94557/79ee6e1c-834c-43ff-8dcc-1385cc20b4c2/9e9e4298-f102-4294-8a71-c71ffc0789bb"
-					(reference "R10")
+					(reference "R23")
+					(unit 1)
+				)
+				(path "/f171b770-6a1a-4d3a-9dbb-25a622b94557/79ee6e1c-834c-43ff-8dcc-1385cc20b4c2/9e9e4298-f102-4294-8a71-c71ffc0789bb"
+					(reference "R25")
 					(unit 1)
 				)
@@
 		(dnp no)
 		(fields_autoplaced yes)
-		(property "Reference" "D7"
+		(property "Reference" "D18"
 			(at 132.08 85.0899 90)
 			(show_name no)
@@
 			(project "PLC4UNI"
 				(path "/f171b770-6a1a-4d3a-9dbb-25a622b94557/79ee6e1c-834c-43ff-8dcc-1385cc20b4c2/1a95a96f-95b5-47d3-8bba-4935d279501e"
-					(reference "D7")
-					(unit 1)
-				)
-				(path "/f171b770-6a1a-4d3a-9dbb-25a622b94557/79ee6e1c-834c-43ff-8dcc-1385cc20b4c2/9e9e4298-f102-4294-8a71-c71ffc0789bb"
-					(reference "D8")
-					(unit 1)
-				)
+					(reference "D18")
+					(unit 1)
+				)
+				(path "/f171b770-6a1a-4d3a-9dbb-25a622b94557/79ee6e1c-834c-43ff-8dcc-1385cc20b4c2/9e9e4298-f102-4294-8a71-c71ffc0789bb"
+					(reference "D20")
+					(unit 1)
+				)
