File: PCB/PLC4UNI/IN-DI.kicad_sch (KiCad schematic)
At the start: 8 parts, among them U5 AT3H4B-CUH-S

Commit message: add ruteo buck-converter, inputs pnp,npn
Parts:
- renumbered C13 to C11, C7 to C12, D9 to D21, R25 to R27, R31 to R28, R19 to R29, R13 to R30, U5 to U9
