File: PCB/PLC4UNI/OUT-4-20MA.kicad_sch (KiCad schematic)
At the start: 11 parts, among them Q1 NCE60P04R, U13 GP8302-TC50-EW

Commit message: add ruteo buck-converter, inputs pnp,npn
Parts:
- renumbered C27 to C31, C28 to C32, C29 to C33, D16 to D28, D17 to D29, D18 to D30, Q1 to Q5, R44 to R58, R45 to R59, R46 to R60, U13 to U17
Changed lines of the file:
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@@
 		(dnp no)
 		(fields_autoplaced yes)
-		(property "Reference" "#PWR040"
+		(property "Reference" "#PWR079"
 			(at 139.7 68.58 0)
 			(hide yes)
@@
 			(project "PLC4UNI"
 				(path "/f171b770-6a1a-4d3a-9dbb-25a622b94557/79ee6e1c-834c-43ff-8dcc-1385cc20b4c2/341047b3-5143-4609-a036-c3108fb9e880"
-					(reference "#PWR040")
+					(reference "#PWR079")
 					(unit 1)
 				)
@@
 		(dnp no)
 		(fields_autoplaced yes)
-		(property "Reference" "#PWR038"
+		(property "Reference" "#PWR076"
 			(at 102.87 106.68 0)
 			(hide yes)
@@
 			(project "PLC4UNI"
 				(path "/f171b770-6a1a-4d3a-9dbb-25a622b94557/79ee6e1c-834c-43ff-8dcc-1385cc20b4c2/341047b3-5143-4609-a036-c3108fb9e880"
-					(reference "#PWR038")
+					(reference "#PWR076")
 					(unit 1)
 				)
@@
 		(dnp no)
 		(fields_autoplaced yes)
-		(property "Reference" "R44"
+		(property "Reference" "R58"
 			(at 71.12 92.7099 0)
 			(show_name no)
@@
 			(project "PLC4UNI"
 				(path "/f171b770-6a1a-4d3a-9dbb-25a622b94557/79ee6e1c-834c-43ff-8dcc-1385cc20b4c2/341047b3-5143-4609-a036-c3108fb9e880"
-					(reference "R44")
+					(reference "R58")
 					(unit 1)
 				)
@@
 		(dnp no)
 		(fields_autoplaced yes)
-		(property "Reference" "D18"
+		(property "Reference" "D30"
 			(at 203.2 90.17 0)
 			(show_name no)
@@
 			(project "PLC4UNI"
 				(path "/f171b770-6a1a-4d3a-9dbb-25a622b94557/79ee6e1c-834c-43ff-8dcc-1385cc20b4c2/341047b3-5143-4609-a036-c3108fb9e880"
-					(reference "D18")
+					(reference "D30")
 					(unit 1)
 				)
@@
 		(dnp no)
 		(fields_autoplaced yes)
-		(property "Reference" "D17"
+		(property "Reference" "D29"
 			(at 176.53 101.5999 90)
 			(show_name no)
@@
 			(project "PLC4UNI"
 				(path "/f171b770-6a1a-4d3a-9dbb-25a622b94557/79ee6e1c-834c-43ff-8dcc-1385cc20b4c2/341047b3-5143-4609-a036-c3108fb9e880"
-					(reference "D17")
+					(reference "D29")
 					(unit 1)
 				)
@@
 		(dnp no)
 		(fields_autoplaced yes)
-		(property "Reference" "#PWR033"
+		(property "Reference" "#PWR072"
 			(at 57.15 76.2 0)
 			(hide yes)
@@
 			(project "PLC4UNI"
 				(path "/f171b770-6a1a-4d3a-9dbb-25a622b94557/79ee6e1c-834c-43ff-8dcc-1385cc20b4c2/341047b3-5143-4609-a036-c3108fb9e880"
-					(reference "#PWR033")
+					(reference "#PWR072")
 					(unit 1)
 				)
@@
 		(dnp no)
 		(fields_autoplaced yes)
-		(property "Reference" "#PWR041"
+		(property "Reference" "#PWR081"
 			(at 173.99 116.84 0)
 			(hide yes)
@@
 			(project "PLC4UNI"
 				(path "/f171b770-6a1a-4d3a-9dbb-25a622b94557/79ee6e1c-834c-43ff-8dcc-1385cc20b4c2/341047b3-5143-4609-a036-c3108fb9e880"
-					(reference "#PWR041")
+					(reference "#PWR081")
 					(unit 1)
 				)
@@
 		(in_pos_files yes)
 		(dnp no)
-		(property "Reference" "R45"
+		(property "Reference" "R59"
 			(at 142.24 101.5999 0)
 			(show_name no)
@@
 			(project "PLC4UNI"
 				(path "/f171b770-6a1a-4d3a-9dbb-25a622b94557/79ee6e1c-834c-43ff-8dcc-1385cc20b4c2/341047b3-5143-4609-a036-c3108fb9e880"
-					(reference "R45")
+					(reference "R59")
 					(unit 1)
 				)
@@
 		(dnp no)
 		(fields_autoplaced yes)
-		(property "Reference" "D16"
+		(property "Reference" "D28"
 			(at 142.24 71.1199 90)
 			(show_name no)
@@
 			(project "PLC4UNI"
 				(path "/f171b770-6a1a-4d3a-9dbb-25a622b94557/79ee6e1c-834c-43ff-8dcc-1385cc20b4c2/341047b3-5143-4609-a036-c3108fb9e880"
-					(reference "D16")
+					(reference "D28")
 					(unit 1)
 				)
@@
 		(dnp no)
 		(fields_autoplaced yes)
-		(property "Reference" "#PWR035"
+		(property "Reference" "#PWR077"
 			(at 107.95 106.68 0)
 			(hide yes)
@@
 			(project "PLC4UNI"
 				(path "/f171b770-6a1a-4d3a-9dbb-25a622b94557/79ee6e1c-834c-43ff-8dcc-1385cc20b4c2/341047b3-5143-4609-a036-c3108fb9e880"
-					(reference "#PWR035")
+					(reference "#PWR077")
 					(unit 1)
 				)
@@
 		(dnp no)
 		(fields_autoplaced yes)
-		(property "Reference" "R46"
+		(property "Reference" "R60"
 			(at 189.23 90.17 90)
 			(show_name no)
@@
 			(project "PLC4UNI"
 				(path "/f171b770-6a1a-4d3a-9dbb-25a622b94557/79ee6e1c-834c-43ff-8dcc-1385cc20b4c2/341047b3-5143-4609-a036-c3108fb9e880"
-					(reference "R46")
+					(reference "R60")
 					(unit 1)
 				)
@@
 		(dnp no)
 		(fields_autoplaced yes)
-		(property "Reference" "#PWR039"
+		(property "Reference" "#PWR080"
 			(at 139.7 116.84 0)
 			(hide yes)
@@
 			(project "PLC4UNI"
 				(path "/f171b770-6a1a-4d3a-9dbb-25a622b94557/79ee6e1c-834c-43ff-8dcc-1385cc20b4c2/341047b3-5143-4609-a036-c3108fb9e880"
-					(reference "#PWR039")
+					(reference "#PWR080")
 					(unit 1)
 				)
@@
 		(in_pos_files yes)
 		(dnp no)
-		(property "Reference" "C27"
+		(property "Reference" "C31"
 			(at 53.34 91.4399 0)
 			(show_name no)
@@
 			(project "PLC4UNI"
 				(path "/f171b770-6a1a-4d3a-9dbb-25a622b94557/79ee6e1c-834c-43ff-8dcc-1385cc20b4c2/341047b3-5143-4609-a036-c3108fb9e880"
-					(reference "C27")
+					(reference "C31")
 					(unit 1)
 				)
@@
 		(dnp no)
 		(fields_autoplaced yes)
-		(property "Reference" "#PWR036"
+		(property "Reference" "#PWR078"
 			(at 134.62 116.84 0)
 			(hide yes)
@@
 			(project "PLC4UNI"
 				(path "/f171b770-6a1a-4d3a-9dbb-25a622b94557/79ee6e1c-834c-43ff-8dcc-1385cc20b4c2/341047b3-5143-4609-a036-c3108fb9e880"
-					(reference "#PWR036")
+					(reference "#PWR078")
 					(unit 1)
 				)
@@
 		(dnp no)
 		(fields_autoplaced yes)
-		(property "Reference" "#PWR034"
+		(property "Reference" "#PWR073"
 			(at 57.15 106.68 0)
 			(hide yes)
@@
 			(project "PLC4UNI"
 				(path "/f171b770-6a1a-4d3a-9dbb-25a622b94557/79ee6e1c-834c-43ff-8dcc-1385cc20b4c2/341047b3-5143-4609-a036-c3108fb9e880"
-					(reference "#PWR034")
+					(reference "#PWR073")
 					(unit 1)
 				)
@@
 		(dnp no)
 		(fields_autoplaced yes)
-		(property "Reference" "#PWR037"
+		(property "Reference" "#PWR074"
 			(at 68.58 106.68 0)
 			(hide yes)
@@
 			(project "PLC4UNI"
 				(path "/f171b770-6a1a-4d3a-9dbb-25a622b94557/79ee6e1c-834c-43ff-8dcc-1385cc20b4c2/341047b3-5143-4609-a036-c3108fb9e880"
-					(reference "#PWR037")
+					(reference "#PWR074")
 					(unit 1)
 				)
@@
 		(in_pos_files yes)
 		(dnp no)
-		(property "Reference" "Q1"
+		(property "Reference" "Q5"
 			(at 154.94 87.6301 0)
 			(show_name no)
@@
 			(project "PLC4UNI"
 				(path "/f171b770-6a1a-4d3a-9dbb-25a622b94557/79ee6e1c-834c-43ff-8dcc-1385cc20b4c2/341047b3-5143-4609-a036-c3108fb9e880"
-					(reference "Q1")
+					(reference "Q5")
 					(unit 1)
 				)
@@
 		(dnp no)
 		(fields_autoplaced yes)
-		(property "Reference" "#PWR042"
+		(property "Reference" "#PWR075"
 			(at 83.82 106.68 0)
 			(hide yes)
@@
 			(project "PLC4UNI"
 				(path "/f171b770-6a1a-4d3a-9dbb-25a622b94557/79ee6e1c-834c-43ff-8dcc-1385cc20b4c2/341047b3-5143-4609-a036-c3108fb9e880"
-					(reference "#PWR042")
+					(reference "#PWR075")
 					(unit 1)
 				)
@@
 		(dnp no)
 		(fields_autoplaced yes)
-		(property "Reference" "U13"
+		(property "Reference" "U17"
 			(at 83.82 68.58 0)
 			(show_name no)
@@
 			(project "PLC4UNI"
 				(path "/f171b770-6a1a-4d3a-9dbb-25a622b94557/79ee6e1c-834c-43ff-8dcc-1385cc20b4c2/341047b3-5143-4609-a036-c3108fb9e880"
-					(reference "U13")
+					(reference "U17")
 					(unit 1)
 				)
@@
 		(in_pos_files yes)
 		(dnp no)
-		(property "Reference" "C28"
+		(property "Reference" "C32"
 			(at 111.76 90.1699 0)
 			(show_name no)
@@
 			(project "PLC4UNI"
 				(path "/f171b770-6a1a-4d3a-9dbb-25a622b94557/79ee6e1c-834c-43ff-8dcc-1385cc20b4c2/341047b3-5143-4609-a036-c3108fb9e880"
-					(reference "C28")
+					(reference "C32")
 					(unit 1)
 				)
@@
 		(in_pos_files yes)
 		(dnp no)
-		(property "Reference" "C29"
+		(property "Reference" "C33"
 			(at 130.81 101.5999 0)
 			(show_name no)
@@
 			(project "PLC4UNI"
 				(path "/f171b770-6a1a-4d3a-9dbb-25a622b94557/79ee6e1c-834c-43ff-8dcc-1385cc20b4c2/341047b3-5143-4609-a036-c3108fb9e880"
-					(reference "C29")
-					(unit 1)
-				)
+					(reference "C33")
+					(unit 1)
+				)
