File: PCB/PLC4UNI/OUT-NPN.kicad_sch (KiCad schematic)
At the start: 3 parts, among them Q2 ZXMS6004FFQTA

Commit message: add ruteo buck-converter, inputs pnp,npn
Parts:
- renumbered D21 to D9, Q2 to Q1, R49 to R11
Changed lines of the file:
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@@
 		(dnp no)
 		(fields_autoplaced yes)
-		(property "Reference" "Q2"
+		(property "Reference" "Q1"
 			(at 138.43 66.04 90)
 			(show_name no)
@@
 			(project "PLC4UNI"
 				(path "/f171b770-6a1a-4d3a-9dbb-25a622b94557/79ee6e1c-834c-43ff-8dcc-1385cc20b4c2/009579de-184b-42e1-8af9-e50d895be0bd"
-					(reference "Q5")
+					(reference "Q4")
 					(unit 1)
 				)
 				(path "/f171b770-6a1a-4d3a-9dbb-25a622b94557/79ee6e1c-834c-43ff-8dcc-1385cc20b4c2/20065da2-17e4-4bca-b0c0-12a2104d40c1"
+					(reference "Q2")
+					(unit 1)
+				)
+				(path "/f171b770-6a1a-4d3a-9dbb-25a622b94557/79ee6e1c-834c-43ff-8dcc-1385cc20b4c2/d7efe19f-e511-4a70-9143-d7b7e8b791cc"
+					(reference "Q1")
+					(unit 1)
+				)
+				(path "/f171b770-6a1a-4d3a-9dbb-25a622b94557/79ee6e1c-834c-43ff-8dcc-1385cc20b4c2/e6d75fc0-930f-48ad-ab92-a65c466950b6"
 					(reference "Q3")
-					(unit 1)
-				)
-				(path "/f171b770-6a1a-4d3a-9dbb-25a622b94557/79ee6e1c-834c-43ff-8dcc-1385cc20b4c2/d7efe19f-e511-4a70-9143-d7b7e8b791cc"
-					(reference "Q2")
-					(unit 1)
-				)
-				(path "/f171b770-6a1a-4d3a-9dbb-25a622b94557/79ee6e1c-834c-43ff-8dcc-1385cc20b4c2/e6d75fc0-930f-48ad-ab92-a65c466950b6"
-					(reference "Q4")
 					(unit 1)
 				)
@@
 		(dnp no)
 		(fields_autoplaced yes)
-		(property "Reference" "D21"
+		(property "Reference" "D9"
 			(at 156.21 65.9764 90)
 			(show_name no)
@@
 			(project "PLC4UNI"
 				(path "/f171b770-6a1a-4d3a-9dbb-25a622b94557/79ee6e1c-834c-43ff-8dcc-1385cc20b4c2/009579de-184b-42e1-8af9-e50d895be0bd"
-					(reference "D24")
+					(reference "D12")
 					(unit 1)
 				)
 				(path "/f171b770-6a1a-4d3a-9dbb-25a622b94557/79ee6e1c-834c-43ff-8dcc-1385cc20b4c2/20065da2-17e4-4bca-b0c0-12a2104d40c1"
-					(reference "D22")
+					(reference "D10")
 					(unit 1)
 				)
 				(path "/f171b770-6a1a-4d3a-9dbb-25a622b94557/79ee6e1c-834c-43ff-8dcc-1385cc20b4c2/d7efe19f-e511-4a70-9143-d7b7e8b791cc"
-					(reference "D21")
+					(reference "D9")
 					(unit 1)
 				)
 				(path "/f171b770-6a1a-4d3a-9dbb-25a622b94557/79ee6e1c-834c-43ff-8dcc-1385cc20b4c2/e6d75fc0-930f-48ad-ab92-a65c466950b6"
-					(reference "D23")
+					(reference "D11")
 					(unit 1)
 				)
@@
 		(dnp no)
 		(fields_autoplaced yes)
-		(property "Reference" "#PWR048"
+		(property "Reference" "#PWR030"
 			(at 123.19 93.98 0)
 			(hide yes)
@@
 			(project "PLC4UNI"
 				(path "/f171b770-6a1a-4d3a-9dbb-25a622b94557/79ee6e1c-834c-43ff-8dcc-1385cc20b4c2/009579de-184b-42e1-8af9-e50d895be0bd"
-					(reference "#PWR054")
+					(reference "#PWR040")
 					(unit 1)
 				)
 				(path "/f171b770-6a1a-4d3a-9dbb-25a622b94557/79ee6e1c-834c-43ff-8dcc-1385cc20b4c2/20065da2-17e4-4bca-b0c0-12a2104d40c1"
-					(reference "#PWR050")
+					(reference "#PWR032")
 					(unit 1)
 				)
 				(path "/f171b770-6a1a-4d3a-9dbb-25a622b94557/79ee6e1c-834c-43ff-8dcc-1385cc20b4c2/d7efe19f-e511-4a70-9143-d7b7e8b791cc"
-					(reference "#PWR048")
+					(reference "#PWR030")
 					(unit 1)
 				)
 				(path "/f171b770-6a1a-4d3a-9dbb-25a622b94557/79ee6e1c-834c-43ff-8dcc-1385cc20b4c2/e6d75fc0-930f-48ad-ab92-a65c466950b6"
-					(reference "#PWR052")
+					(reference "#PWR034")
 					(unit 1)
 				)
@@
 		(dnp no)
 		(fields_autoplaced yes)
-		(property "Reference" "R49"
+		(property "Reference" "R11"
 			(at 156.21 57.1499 0)
 			(show_name no)
@@
 			(project "PLC4UNI"
 				(path "/f171b770-6a1a-4d3a-9dbb-25a622b94557/79ee6e1c-834c-43ff-8dcc-1385cc20b4c2/009579de-184b-42e1-8af9-e50d895be0bd"
-					(reference "R52")
+					(reference "R14")
 					(unit 1)
 				)
 				(path "/f171b770-6a1a-4d3a-9dbb-25a622b94557/79ee6e1c-834c-43ff-8dcc-1385cc20b4c2/20065da2-17e4-4bca-b0c0-12a2104d40c1"
-					(reference "R50")
+					(reference "R12")
 					(unit 1)
 				)
 				(path "/f171b770-6a1a-4d3a-9dbb-25a622b94557/79ee6e1c-834c-43ff-8dcc-1385cc20b4c2/d7efe19f-e511-4a70-9143-d7b7e8b791cc"
-					(reference "R49")
+					(reference "R11")
 					(unit 1)
 				)
 				(path "/f171b770-6a1a-4d3a-9dbb-25a622b94557/79ee6e1c-834c-43ff-8dcc-1385cc20b4c2/e6d75fc0-930f-48ad-ab92-a65c466950b6"
-					(reference "R51")
+					(reference "R13")
 					(unit 1)
 				)
@@
 		(in_pos_files yes)
 		(dnp no)
-		(property "Reference" "#PWR049"
+		(property "Reference" "#PWR031"
 			(at 153.67 54.61 0)
 			(hide yes)
@@
 			(project "PLC4UNI"
 				(path "/f171b770-6a1a-4d3a-9dbb-25a622b94557/79ee6e1c-834c-43ff-8dcc-1385cc20b4c2/009579de-184b-42e1-8af9-e50d895be0bd"
-					(reference "#PWR055")
+					(reference "#PWR041")
 					(unit 1)
 				)
 				(path "/f171b770-6a1a-4d3a-9dbb-25a622b94557/79ee6e1c-834c-43ff-8dcc-1385cc20b4c2/20065da2-17e4-4bca-b0c0-12a2104d40c1"
-					(reference "#PWR051")
+					(reference "#PWR033")
 					(unit 1)
 				)
 				(path "/f171b770-6a1a-4d3a-9dbb-25a622b94557/79ee6e1c-834c-43ff-8dcc-1385cc20b4c2/d7efe19f-e511-4a70-9143-d7b7e8b791cc"
-					(reference "#PWR049")
+					(reference "#PWR031")
 					(unit 1)
 				)
 				(path "/f171b770-6a1a-4d3a-9dbb-25a622b94557/79ee6e1c-834c-43ff-8dcc-1385cc20b4c2/e6d75fc0-930f-48ad-ab92-a65c466950b6"
-					(reference "#PWR053")
-					(unit 1)
-				)
+					(reference "#PWR035")
+					(unit 1)
+				)
