File: PCB/PLC4UNI/OUT-PNP.kicad_sch (KiCad schematic)
At the start: 5 parts, among them U14 BTS723GWXUMA1

Commit message: add ruteo buck-converter, inputs pnp,npn
Parts:
- renumbered D19 to D7, D20 to D8, R48 to R10, R47 to R9, U14 to U7
Changed lines of the file:
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@@
 		(dnp no)
 		(fields_autoplaced yes)
-		(property "Reference" "U14"
+		(property "Reference" "U7"
 			(at 140.97 62.23 0)
 			(show_name no)
@@
 			(project "PLC4UNI"
 				(path "/f171b770-6a1a-4d3a-9dbb-25a622b94557/79ee6e1c-834c-43ff-8dcc-1385cc20b4c2/2dccfd7b-69f0-4b97-a6e1-c1e412fa5c14"
-					(reference "U14")
+					(reference "U7")
 					(unit 1)
 				)
@@
 		(dnp no)
 		(fields_autoplaced yes)
-		(property "Reference" "D20"
+		(property "Reference" "D8"
 			(at 179.0065 116.84 0)
 			(show_name no)
@@
 			(project "PLC4UNI"
 				(path "/f171b770-6a1a-4d3a-9dbb-25a622b94557/79ee6e1c-834c-43ff-8dcc-1385cc20b4c2/2dccfd7b-69f0-4b97-a6e1-c1e412fa5c14"
-					(reference "D20")
+					(reference "D8")
 					(unit 1)
 				)
@@
 		(dnp no)
 		(fields_autoplaced yes)
-		(property "Reference" "R47"
+		(property "Reference" "R9"
 			(at 168.91 80.01 90)
 			(show_name no)
@@
 			(project "PLC4UNI"
 				(path "/f171b770-6a1a-4d3a-9dbb-25a622b94557/79ee6e1c-834c-43ff-8dcc-1385cc20b4c2/2dccfd7b-69f0-4b97-a6e1-c1e412fa5c14"
-					(reference "R47")
+					(reference "R9")
 					(unit 1)
 				)
@@
 		(dnp no)
 		(fields_autoplaced yes)
-		(property "Reference" "#PWR046"
+		(property "Reference" "#PWR028"
 			(at 186.69 95.25 0)
 			(hide yes)
@@
 			(project "PLC4UNI"
 				(path "/f171b770-6a1a-4d3a-9dbb-25a622b94557/79ee6e1c-834c-43ff-8dcc-1385cc20b4c2/2dccfd7b-69f0-4b97-a6e1-c1e412fa5c14"
-					(reference "#PWR046")
+					(reference "#PWR028")
 					(unit 1)
 				)
@@
 		(dnp no)
 		(fields_autoplaced yes)
-		(property "Reference" "#PWR043"
+		(property "Reference" "#PWR026"
 			(at 118.11 72.39 0)
 			(hide yes)
@@
 			(project "PLC4UNI"
 				(path "/f171b770-6a1a-4d3a-9dbb-25a622b94557/79ee6e1c-834c-43ff-8dcc-1385cc20b4c2/2dccfd7b-69f0-4b97-a6e1-c1e412fa5c14"
-					(reference "#PWR043")
+					(reference "#PWR026")
 					(unit 1)
 				)
@@
 		(dnp no)
 		(fields_autoplaced yes)
-		(property "Reference" "#PWR044"
+		(property "Reference" "#PWR027"
 			(at 158.75 80.01 0)
 			(hide yes)
@@
 			(project "PLC4UNI"
 				(path "/f171b770-6a1a-4d3a-9dbb-25a622b94557/79ee6e1c-834c-43ff-8dcc-1385cc20b4c2/2dccfd7b-69f0-4b97-a6e1-c1e412fa5c14"
-					(reference "#PWR044")
+					(reference "#PWR027")
 					(unit 1)
 				)
@@
 		(dnp no)
 		(fields_autoplaced yes)
-		(property "Reference" "#PWR045"
+		(property "Reference" "#PWR025"
 			(at 113.03 72.39 0)
 			(hide yes)
@@
 			(project "PLC4UNI"
 				(path "/f171b770-6a1a-4d3a-9dbb-25a622b94557/79ee6e1c-834c-43ff-8dcc-1385cc20b4c2/2dccfd7b-69f0-4b97-a6e1-c1e412fa5c14"
-					(reference "#PWR045")
+					(reference "#PWR025")
 					(unit 1)
 				)
@@
 		(dnp no)
 		(fields_autoplaced yes)
-		(property "Reference" "D19"
+		(property "Reference" "D7"
 			(at 179.0065 80.01 0)
 			(show_name no)
@@
 			(project "PLC4UNI"
 				(path "/f171b770-6a1a-4d3a-9dbb-25a622b94557/79ee6e1c-834c-43ff-8dcc-1385cc20b4c2/2dccfd7b-69f0-4b97-a6e1-c1e412fa5c14"
-					(reference "D19")
+					(reference "D7")
 					(unit 1)
 				)
@@
 		(dnp no)
 		(fields_autoplaced yes)
-		(property "Reference" "R48"
+		(property "Reference" "R10"
 			(at 168.91 116.84 90)
 			(show_name no)
@@
 			(project "PLC4UNI"
 				(path "/f171b770-6a1a-4d3a-9dbb-25a622b94557/79ee6e1c-834c-43ff-8dcc-1385cc20b4c2/2dccfd7b-69f0-4b97-a6e1-c1e412fa5c14"
-					(reference "R48")
+					(reference "R10")
 					(unit 1)
 				)
@@
 		(dnp no)
 		(fields_autoplaced yes)
-		(property "Reference" "#PWR047"
+		(property "Reference" "#PWR029"
 			(at 186.69 101.6 0)
 			(hide yes)
@@
 			(project "PLC4UNI"
 				(path "/f171b770-6a1a-4d3a-9dbb-25a622b94557/79ee6e1c-834c-43ff-8dcc-1385cc20b4c2/2dccfd7b-69f0-4b97-a6e1-c1e412fa5c14"
-					(reference "#PWR047")
-					(unit 1)
-				)
+					(reference "#PWR029")
+					(unit 1)
+				)
