File: PCB/PLC4UNI/RS485.kicad_sch (KiCad schematic)
At the start: 8 parts, among them U23 TD301M485_C5451847

Commit message: add ruteo buck-converter, inputs pnp,npn
Parts:
- renumbered D30 to D35, D29 to D36, D31 to D37, R70 to R75, R71 to R76, R72 to R77, R73 to R78
Changed lines of the file:
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@@
 		(dnp no)
 		(fields_autoplaced yes)
-		(property "Reference" "#PWR098"
+		(property "Reference" "#PWR0112"
 			(at 168.91 143.51 0)
 			(hide yes)
@@
 			(project "PLC4UNI"
 				(path "/f171b770-6a1a-4d3a-9dbb-25a622b94557/79ee6e1c-834c-43ff-8dcc-1385cc20b4c2/d4e7a445-33fa-42af-97b4-3f58f68ece03"
-					(reference "#PWR098")
+					(reference "#PWR0112")
 					(unit 1)
 				)
@@
 		(dnp no)
 		(fields_autoplaced yes)
-		(property "Reference" "#PWR097"
+		(property "Reference" "#PWR0111"
 			(at 168.91 111.76 0)
 			(hide yes)
@@
 			(project "PLC4UNI"
 				(path "/f171b770-6a1a-4d3a-9dbb-25a622b94557/79ee6e1c-834c-43ff-8dcc-1385cc20b4c2/d4e7a445-33fa-42af-97b4-3f58f68ece03"
-					(reference "#PWR097")
+					(reference "#PWR0111")
 					(unit 1)
 				)
@@
 		(in_pos_files yes)
 		(dnp no)
-		(property "Reference" "R70"
+		(property "Reference" "R75"
 			(at 152.4 118.1099 0)
 			(show_name no)
@@
 			(project "PLC4UNI"
 				(path "/f171b770-6a1a-4d3a-9dbb-25a622b94557/79ee6e1c-834c-43ff-8dcc-1385cc20b4c2/d4e7a445-33fa-42af-97b4-3f58f68ece03"
-					(reference "R70")
+					(reference "R75")
 					(unit 1)
 				)
@@
 		(dnp no)
 		(fields_autoplaced yes)
-		(property "Reference" "D31"
+		(property "Reference" "D37"
 			(at 234.95 137.1599 90)
 			(show_name no)
@@
 			(project "PLC4UNI"
 				(path "/f171b770-6a1a-4d3a-9dbb-25a622b94557/79ee6e1c-834c-43ff-8dcc-1385cc20b4c2/d4e7a445-33fa-42af-97b4-3f58f68ece03"
-					(reference "D31")
+					(reference "D37")
 					(unit 1)
 				)
@@
 		(in_pos_files yes)
 		(dnp no)
-		(property "Reference" "R72"
+		(property "Reference" "R77"
 			(at 248.92 116.8399 0)
 			(show_name no)
@@
 			(project "PLC4UNI"
 				(path "/f171b770-6a1a-4d3a-9dbb-25a622b94557/79ee6e1c-834c-43ff-8dcc-1385cc20b4c2/d4e7a445-33fa-42af-97b4-3f58f68ece03"
-					(reference "R72")
+					(reference "R77")
 					(unit 1)
 				)
@@
 		(in_pos_files yes)
 		(dnp no)
-		(property "Reference" "R73"
+		(property "Reference" "R78"
 			(at 248.92 135.8899 0)
 			(show_name no)
@@
 			(project "PLC4UNI"
 				(path "/f171b770-6a1a-4d3a-9dbb-25a622b94557/79ee6e1c-834c-43ff-8dcc-1385cc20b4c2/d4e7a445-33fa-42af-97b4-3f58f68ece03"
-					(reference "R73")
+					(reference "R78")
 					(unit 1)
 				)
@@
 		(in_pos_files yes)
 		(dnp no)
-		(property "Reference" "R71"
+		(property "Reference" "R76"
 			(at 160.02 118.1099 0)
 			(show_name no)
@@
 			(project "PLC4UNI"
 				(path "/f171b770-6a1a-4d3a-9dbb-25a622b94557/79ee6e1c-834c-43ff-8dcc-1385cc20b4c2/d4e7a445-33fa-42af-97b4-3f58f68ece03"
-					(reference "R71")
+					(reference "R76")
 					(unit 1)
 				)
@@
 		(dnp no)
 		(fields_autoplaced yes)
-		(property "Reference" "D29"
+		(property "Reference" "D36"
 			(at 223.52 113.03 0)
 			(show_name no)
@@
 			(project "PLC4UNI"
 				(path "/f171b770-6a1a-4d3a-9dbb-25a622b94557/79ee6e1c-834c-43ff-8dcc-1385cc20b4c2/d4e7a445-33fa-42af-97b4-3f58f68ece03"
-					(reference "D29")
+					(reference "D36")
 					(unit 1)
 				)
@@
 		(in_pos_files yes)
 		(dnp no)
-		(property "Reference" "D30"
+		(property "Reference" "D35"
 			(at 213.36 137.1599 90)
 			(show_name no)
@@
 			(project "PLC4UNI"
 				(path "/f171b770-6a1a-4d3a-9dbb-25a622b94557/79ee6e1c-834c-43ff-8dcc-1385cc20b4c2/d4e7a445-33fa-42af-97b4-3f58f68ece03"
-					(reference "D30")
-					(unit 1)
-				)
+					(reference "D35")
+					(unit 1)
+				)
