File: PCB/PLC4UNI/ENERGY-METER.kicad_sch (KiCad schematic)
At the start: 26 parts, among them U20 B0303S-1WR3_C7465185, U21 BL0942, U22 ISO7021DR

Commit message: add ruteo buck-converter, inputs pnp,npn
Parts:
- renumbered C39 to C34, C40 to C35, C41 to C36, C43 to C37, C44 to C38, C42 to C39, R56 to R61, R57 to R62, R60 to R63, R58 to R64, R59 to R65, R61 to R66, R62 to R67, R63 to R68, R64 to R69, R65 to R70, R68 to R71, R69 to R72, R66 to R73, R67 to R74, TP9 to TP5, TP10 to TP6, TP8 to TP7, U21 to U18, U20 to U19, U22 to U20

Commit message: power supply and inputs routed
Parts:
- TP5, TP6, TP7: footprint TestPoint:TestPoint_Pad_D4.0mm -> TestPoint:TestPoint_THTPad_D1.5mm_Drill0.7mm
Changed lines of the file:
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@@
 			)
 		)
-		(property "Footprint" "TestPoint:TestPoint_Pad_D4.0mm"
+		(property "Footprint" "TestPoint:TestPoint_THTPad_D1.5mm_Drill0.7mm"
 			(at 128.27 127 0)
 			(hide yes)
@@
 			)
 		)
-		(property "Footprint" "TestPoint:TestPoint_Pad_D4.0mm"
+		(property "Footprint" "TestPoint:TestPoint_THTPad_D1.5mm_Drill0.7mm"
 			(at 196.85 80.01 0)
 			(hide yes)
@@
 			)
 		)
-		(property "Footprint" "TestPoint:TestPoint_Pad_D4.0mm"
+		(property "Footprint" "TestPoint:TestPoint_THTPad_D1.5mm_Drill0.7mm"
 			(at 120.65 154.94 0)
 			(hide yes)
