File: PCB/PLC4UNI/TLY.kicad_sch (KiCad schematic)
At the start: 3 parts, among them K1 G5V-1-DC3, K2 G5V-1-DC3, U15 LK1802

Commit message: add ruteo buck-converter, inputs pnp,npn
Parts:
- renumbered K2 to K1, K1 to K2, U15 to U8
Changed lines of the file:
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@@
 		(dnp no)
 		(fields_autoplaced yes)
-		(property "Reference" "#PWR058"
+		(property "Reference" "#PWR038"
 			(at 172.72 66.04 0)
 			(hide yes)
@@
 			(project "PLC4UNI"
 				(path "/f171b770-6a1a-4d3a-9dbb-25a622b94557/79ee6e1c-834c-43ff-8dcc-1385cc20b4c2/df61efe4-a923-4526-ba02-7b2f723784ab"
-					(reference "#PWR058")
+					(reference "#PWR038")
 					(unit 1)
 				)
@@
 		(dnp no)
 		(fields_autoplaced yes)
-		(property "Reference" "#PWR059"
+		(property "Reference" "#PWR039"
 			(at 177.8 104.14 0)
 			(hide yes)
@@
 			(project "PLC4UNI"
 				(path "/f171b770-6a1a-4d3a-9dbb-25a622b94557/79ee6e1c-834c-43ff-8dcc-1385cc20b4c2/df61efe4-a923-4526-ba02-7b2f723784ab"
-					(reference "#PWR059")
+					(reference "#PWR039")
 					(unit 1)
 				)
@@
 		(in_pos_files yes)
 		(dnp no)
-		(property "Reference" "U15"
+		(property "Reference" "U8"
 			(at 149.86 86.36 0)
 			(show_name no)
@@
 			(project "PLC4UNI"
 				(path "/f171b770-6a1a-4d3a-9dbb-25a622b94557/79ee6e1c-834c-43ff-8dcc-1385cc20b4c2/df61efe4-a923-4526-ba02-7b2f723784ab"
-					(reference "U15")
+					(reference "U8")
 					(unit 1)
 				)
@@
 		(in_pos_files yes)
 		(dnp no)
-		(property "Reference" "K1"
+		(property "Reference" "K2"
 			(at 196.85 112.5199 0)
 			(show_name no)
@@
 			(project "PLC4UNI"
 				(path "/f171b770-6a1a-4d3a-9dbb-25a622b94557/79ee6e1c-834c-43ff-8dcc-1385cc20b4c2/df61efe4-a923-4526-ba02-7b2f723784ab"
-					(reference "K1")
+					(reference "K2")
 					(unit 1)
 				)
@@
 		(dnp no)
 		(fields_autoplaced yes)
-		(property "Reference" "#PWR057"
+		(property "Reference" "#PWR037"
 			(at 138.43 111.76 0)
 			(hide yes)
@@
 			(project "PLC4UNI"
 				(path "/f171b770-6a1a-4d3a-9dbb-25a622b94557/79ee6e1c-834c-43ff-8dcc-1385cc20b4c2/df61efe4-a923-4526-ba02-7b2f723784ab"
-					(reference "#PWR057")
+					(reference "#PWR037")
 					(unit 1)
 				)
@@
 		(in_pos_files yes)
 		(dnp no)
-		(property "Reference" "K2"
+		(property "Reference" "K1"
 			(at 191.77 74.4199 0)
 			(show_name no)
@@
 			(project "PLC4UNI"
 				(path "/f171b770-6a1a-4d3a-9dbb-25a622b94557/79ee6e1c-834c-43ff-8dcc-1385cc20b4c2/df61efe4-a923-4526-ba02-7b2f723784ab"
-					(reference "K2")
+					(reference "K1")
 					(unit 1)
 				)
@@
 		(dnp no)
 		(fields_autoplaced yes)
-		(property "Reference" "#PWR056"
+		(property "Reference" "#PWR036"
 			(at 138.43 86.36 0)
 			(hide yes)
@@
 			(project "PLC4UNI"
 				(path "/f171b770-6a1a-4d3a-9dbb-25a622b94557/79ee6e1c-834c-43ff-8dcc-1385cc20b4c2/df61efe4-a923-4526-ba02-7b2f723784ab"
-					(reference "#PWR056")
+					(reference "#PWR036")
 					(unit 1)
 				)

Commit message: ruteo terminado
Connections:
- net at U8.1 (1C): now also K2.9; no longer K1.9
- net at U8.6 (2C): now also K1.9; no longer K2.9
Changed lines of the file:
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@@
+	(wire
+		(pts
+			(xy 161.29 127) (xy 161.29 90.17)
+		)
+		(stroke
+			(width 0)
+			(type default)
+		)
+	)
 	(wire
 		(pts
@@
 	(wire
 		(pts
-			(xy 172.72 82.55) (xy 172.72 90.17)
+			(xy 158.75 90.17) (xy 161.29 90.17)
+		)
+		(stroke
+			(width 0)
+			(type default)
+		)
+	)
+	(wire
+		(pts
+			(xy 172.72 82.55) (xy 172.72 99.06)
 		)
 		(stroke
@@
 	(wire
 		(pts
-			(xy 161.29 99.06) (xy 161.29 127)
-		)
-		(stroke
-			(width 0)
-			(type default)
-		)
-	)
-	(wire
-		(pts
 			(xy 177.8 120.65) (xy 177.8 127)
 		)
@@
 	(wire
 		(pts
-			(xy 158.75 99.06) (xy 161.29 99.06)
+			(xy 158.75 99.06) (xy 172.72 99.06)
 		)
 		(stroke
@@
 		)
 		(stroke
-			(width 0)
-			(type default)
-		)
-	)
-	(wire
-		(pts
-			(xy 172.72 90.17) (xy 158.75 90.17)
-		)
-		(stroke
